File: pcb/mcu_integration.kicad_pcb (KiCad board)
At the start: 4 copper layers, 90.2 x 95.9 mm, 108 parts, among them IC1 TL7660IDGKR, IC10 AD844_OPAMP_MEL, IC2 TL081IDT, IC3 FOD814_OPTO_NOSHD, IC4 UA78M33CDCYG3, IC5 FOD814_OPTO_MEL, IC6 AD844_OPAMP_AL, IC7 FOD814_OPTO_AL, IC8 AD844_OPAMP_NOSHD, J1 Micro_SD_Card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

Commit message: bare mcu implementation
Parts:
- removed C12, C13, C22, C23, C24: 10u, capstone:T495D
- removed C14, C15, C19, C20, C28, C32, C34, C38, C41: 0.1u, capstone:CAPC220145_88N_KEM-0.1u
- removed C16: 0.01u, capstone:CAPC220145_88N_KEM-0.1u
- removed C17, C18, C43: 0.01u, capstone:C0805
- removed C21, C31, C37: 1u, capstone:C0805-1u
- removed C27: 100n, Capacitor_SMD:C_0402_1005Metric
- removed C29, C30, C35, C36, C39, C40: 0.22u, capstone:C0805-0.22u
- removed C33: 1u, Capacitor_SMD:C_0402_1005Metric
- removed C42: 150u, capstone:CAPC3225X280N_150U
- removed IC1: TL7660IDGKR, capstone:SOP65P490X110-8N-actual
- removed IC10: AD844_OPAMP_MEL, capstone:SOIC127P1032X265-16N-AD844
- removed IC2: TL081IDT, capstone:SOIC127P600X175-8N
- removed IC3: FOD814_OPTO_NOSHD, capstone:SOP254P1016X385-4N-FOD
- removed IC5: FOD814_OPTO_MEL, capstone:SOP254P1016X385-4N-FOD
- removed IC6: AD844_OPAMP_AL, capstone:SOIC127P1032X265-16N-AD844
- removed IC7: FOD814_OPTO_AL, capstone:SOP254P1016X385-4N-FOD
- removed IC8: AD844_OPAMP_NOSHD, capstone:SOIC127P1032X265-16N-AD844
- removed J1: Micro_SD_Card, capstone:22017781
- removed J2, J3: ESQ-126-39-L-D, capstone:ESQ-126-Y-X-D
- removed J_AD844: Conn_01x04, Connector_PinHeader_2.54mm:PinHeader_1x04_P2.54mm_Vertical
- removed J_FOD814: Conn_01x06, Connector_PinHeader_2.54mm:PinHeader_1x06_P2.54mm_Vertical
- removed J_REF192, J_SIG1: Conn_01x03, Connector_PinHeader_2.54mm:PinHeader_1x03_P2.54mm_Vertical
- removed R10: 1.0k, Resistor_SMD:R_0402_1005Metric
- removed R11, R9: 1.8k, Resistor_SMD:R_0402_1005Metric
- removed R12: 330, Resistor_SMD:R_0402_1005Metric
- removed R13: 12k, Resistor_SMD:R_0402_1005Metric
- removed R14, R32: 56k, Resistor_SMD:R_0402_1005Metric
- removed R15, R19, R23, R33: 200, Resistor_SMD:R_0402_1005Metric
- removed R16, R20, R24: 47, Resistor_SMD:R_0402_1005Metric
- removed R17, R18, R26, R27, R29, R30: 100, Resistor_SMD:R_0402_1005Metric
- removed R21: 150k, Resistor_SMD:R_0402_1005Metric
- removed R22, R28, R34, R5, R6, R8: 100k, Resistor_SMD:R_0402_1005Metric
- removed R25, R31, R35: 1k, Resistor_SMD:R_0402_1005Metric
- removed R3, R4: 2.2k, Resistor_SMD:R_0402_1005Metric
- removed R7: 220k, Resistor_SMD:R_0402_1005Metric
- removed U2: REF192_NOSHD, capstone:R_8_ADI-REF
- removed U3: REF192_AL, capstone:R_8_ADI-REF
- removed U4: REF192_MEL, capstone:R_8_ADI-REF
- removed U5: TPS2069CDBVR_MOSFET, capstone:DBV5_TEX_MF
- added J_PWR1: Conn_01x06, Connector_PinHeader_2.54mm:PinHeader_1x06_P2.54mm_Vertical, F.Cu at (158.5, 93.0)
Connections:
- C1 pad 1: 3.3V Output -> +3.3V
- C2 pad 1: 3.3V Output -> +3.3V
- C25 pad 1: /Evan -5V and signal gen/+5V_EXT -> +5V
- C26 pad 1: 3.3V Output -> +3.3V
- C3 pad 1: 3.3V Output -> +3.3V
- C4 pad 1: 3.3V Output -> +3.3V
- C5 pad 1: 3.3V Output -> +3.3V
- C8 pad 1: 3.3V Output -> +3.3V
- FB1 pad 2: 3.3V Output -> +3.3V
- IC4 pad 1: /Evan -5V and signal gen/+5V_EXT -> +5V
- IC4 pad 3: 3.3V Output -> +3.3V
- U1 pad 1: 3.3V Output -> +3.3V
- U1 pad 10: ADC1_IN12_OPTO_F_MEL -> unconnected-(U1-PC2-Pad10)
- U1 pad 11: ADC1_IN13_OPTO_E_MEL -> unconnected-(U1-PC3-Pad11)
- U1 pad 14: ADC1_IN0_SINE -> unconnected-(U1-PA0-Pad14)
- U1 pad 15: ADC1_IN1_OPAMP_NOSHD -> unconnected-(U1-PA1-Pad15)
- U1 pad 16: ADC1_IN2_OPAMP_MEL -> unconnected-(U1-PA2-Pad16)
- U1 pad 17: ADC1_IN3_OPAMP_AL -> unconnected-(U1-PA3-Pad17)
- U1 pad 19: 3.3V Output -> +3.3V
- U1 pad 20: ADC1_IN4_VREF_NOSHD -> unconnected-(U1-PA4-Pad20)
- U1 pad 21: ADC1_IN5_VREF_MEL -> unconnected-(U1-PA5-Pad21)
- U1 pad 22: ADC1_IN6_VREF_AL -> unconnected-(U1-PA6-Pad22)
- U1 pad 23: ADC1_IN7_VREG_NOSHD -> unconnected-(U1-PA7-Pad23)
- U1 pad 24: ADC1_IN14_OPTO_F_AL -> unconnected-(U1-PC4-Pad24)
- U1 pad 25: ADC1_IN15_OPTO_E_AL -> unconnected-(U1-PC5-Pad25)
- U1 pad 26: ADC1_IN8_VREG_MEL -> unconnected-(U1-PB0-Pad26)
- U1 pad 27: ADC1_IN9_VREG_AL -> unconnected-(U1-PB1-Pad27)
- U1 pad 32: 3.3V Output -> +3.3V
- U1 pad 33: /SPI2_CS_NSS -> unconnected-(U1-PB12-Pad33)
- U1 pad 34: /SPI2_SCK -> unconnected-(U1-PB13-Pad34)
- U1 pad 35: /SPI2_MISO -> unconnected-(U1-PB14-Pad35)
- U1 pad 36: /SPI2_MOSI -> unconnected-(U1-PB15-Pad36)
- U1 pad 37: MOSFET_CONTROL -> unconnected-(U1-PC6-Pad37)
- U1 pad 38: SIG_SQUARE -> unconnected-(U1-PC7-Pad38)
- U1 pad 48: 3.3V Output -> +3.3V
- U1 pad 58: OBC_I2C_SCL -> unconnected-(U1-PB6-Pad58)
- U1 pad 59: OBC_I2C_SDA -> unconnected-(U1-PB7-Pad59)
- U1 pad 64: 3.3V Output -> +3.3V
- U1 pad 8: ADC1_IN10_OPTO_F_NOSHD -> unconnected-(U1-PC0-Pad8)
- U1 pad 9: ADC1_IN11_OPTO_E_NOSHD -> unconnected-(U1-PC1-Pad9)
Routing:
- net ADC1_IN0_SINE: track 200.7 -> 0.00 mm, vias 3 -> 0
- net 3.3V Output: track 147.5 -> 0.32 mm
- net -5V Output: track 140.1 -> 0.00 mm
- net /Evan -5V and signal gen/+5V_EXT: track 102.6 -> 0.00 mm
- net +3.3V: track 0.00 -> 94.4 mm
- net ADC1_IN3_OPAMP_AL: track 88.8 -> 0.00 mm
- net ADC1_IN10_OPTO_F_NOSHD: track 86.7 -> 0.00 mm, vias 2 -> 0
- net ADC1_IN13_OPTO_E_MEL: track 68.7 -> 0.00 mm, vias 2 -> 0
- net ADC1_IN2_OPAMP_MEL: track 67.9 -> 0.00 mm, vias 2 -> 0
- net +5V: track 91.8 -> 33.2 mm, vias 15 -> 0
- net ADC1_IN15_OPTO_E_AL: track 56.4 -> 0.00 mm, vias 2 -> 0
- net ADC1_IN1_OPAMP_NOSHD: track 55.4 -> 0.00 mm, vias 2 -> 0
- net ADC1_IN14_OPTO_F_AL: track 54.1 -> 0.00 mm, vias 2 -> 0
- net ADC1_IN12_OPTO_F_MEL: track 53.3 -> 0.00 mm
- net /SPI2_MISO: track 44.5 -> 0.00 mm
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Other:
- board text removed: "AL"
- board text removed: "CUBICS Analog IC Shielding Payload Karim A., Evan C., Matthew H. REV B March 8th, 2024"
- board text removed: "E_AL"
- board text removed: "E_MEL"
- board text removed: "E_NOSHD"
- board text removed: "FORMAT AS FAT!"
- board text removed: "F_AL"
- board text removed: "F_MEL"
- board text removed: "F_NOSHD"
- board text removed: "MEL"
- board text removed: "NOSHD"
- board text removed: "SINE"
- board text removed: "SQ_LP"
- board text removed: "WB"
- board text removed: "https://github.com/kaitallaoua/capstone-pcb https://github.com/kaitallaoua/capstone-cubeide"
