File: pcb/mcu_integration.kicad_sch (KiCad schematic)
At the start: 28 parts, among them J1 Micro_SD_Card, U1 STM32F103RBTx, Y1 ECS-80-18-5PX-GM-TR

Commit message: bare mcu implementation
Parts:
- removed C27: 100n, Capacitor_SMD:C_0402_1005Metric, symbol Device:C
- removed C33: 1u, Capacitor_SMD:C_0402_1005Metric, symbol Device:C
- removed J1: Micro_SD_Card, capstone:22017781, symbol capstone:2201778-1
- removed R3, R4: 2.2k, Resistor_SMD:R_0402_1005Metric, symbol Device:R
- added C25: 0.33u, capstone:C0805, symbol capstone:C0805C334K3RACAUTO7210
- added C26: 0.1u, capstone:CAPC220145_88N_KEM-0.1u, symbol capstone:C0805C104K5RAC7210
- added IC4: UA78M33CDCYG3, capstone:SOT230P700X180-4N, symbol capstone:UA78M33CDCYG3
- added J_PWR1: Conn_01x06, Connector_PinHeader_2.54mm:PinHeader_1x06_P2.54mm_Vertical, symbol Connector_Generic:Conn_01x06
Connections:
- net 3.3V Output: no longer C1.1, C2.1, C3.1, C4.1, C5.1, C8.1, FB1.2, U1.1 (VBAT), U1.19 (VDD), U1.32 (VDD), U1.48 (VDD), U1.64 (VDD)
- net GND: now also C25.2, C26.2, IC4.2 (COMMON_1), J_PWR1.1 (Pin_1), J_PWR1.2 (Pin_2)
- net ADC1_IN0_SINE: no longer names the net of U1.14 (PA0)
- net ADC1_IN10_OPTO_F_NOSHD: no longer names the net of U1.8 (PC0)
- net ADC1_IN11_OPTO_E_NOSHD: no longer names the net of U1.9 (PC1)
- net ADC1_IN12_OPTO_F_MEL: no longer names the net of U1.10 (PC2)
- net ADC1_IN13_OPTO_E_MEL: no longer names the net of U1.11 (PC3)
- net ADC1_IN14_OPTO_F_AL: no longer names the net of U1.24 (PC4)
- net ADC1_IN15_OPTO_E_AL: no longer names the net of U1.25 (PC5)
- net ADC1_IN1_OPAMP_NOSHD: no longer names the net of U1.15 (PA1)
- net ADC1_IN2_OPAMP_MEL: no longer names the net of U1.16 (PA2)
- net ADC1_IN3_OPAMP_AL: no longer names the net of U1.17 (PA3)
- net ADC1_IN4_VREF_NOSHD: no longer names the net of U1.20 (PA4)
- net ADC1_IN5_VREF_MEL: no longer names the net of U1.21 (PA5)
- net ADC1_IN6_VREF_AL: no longer names the net of U1.22 (PA6)
- net ADC1_IN7_VREG_NOSHD: no longer names the net of U1.23 (PA7)
- net ADC1_IN8_VREG_MEL: no longer names the net of U1.26 (PB0)
- net ADC1_IN9_VREG_AL: no longer names the net of U1.27 (PB1)
- net MOSFET_CONTROL: no longer names the net of U1.37 (PC6)
- net OBC_I2C_SCL: no longer names the net of U1.58 (PB6)
- net OBC_I2C_SDA: no longer names the net of U1.59 (PB7)
- net SIG_SQUARE: no longer names the net of U1.38 (PC7)
- net SPI2_CS_NSS: no longer names the net of U1.33 (PB12)
- net SPI2_MISO: no longer names the net of U1.35 (PB14)
- net SPI2_MOSI: no longer names the net of U1.36 (PB15)
- net SPI2_SCK: no longer names the net of U1.34 (PB13)
- new net +3.3V: C1.1, C2.1, C26.1, C3.1, C4.1, C5.1, C8.1, FB1.2, IC4.3 (OUTPUT), U1.1 (VBAT), U1.19 (VDD), U1.32 (VDD), U1.48 (VDD), U1.64 (VDD)
- new net +5V: C25.1, IC4.1 (INPUT), J_PWR1.5 (Pin_5), J_PWR1.6 (Pin_6)
- no-connect marks 26 -> 25
Other:
- removed sheet Evan -5V and signal gen
- removed sheet Matt IC Tests
- title: Regina Payload Cubesat MCU Integration -> Robot Pcb
